Commit message: Semi-Functional Eve URDF

File: urdf/eve.urdf (robot description, URDF)
Before this commit: robot eve, 4 links, 3 joints
Links:
- added link left_arm_x
- added link left_arm_y
- added link left_arm_z
- added link right_arm_x
- added link right_arm_y
- added link right_arm_z
- link left_arm: geometry visual box size=0.5 0.2 0.01
- link right_arm: geometry visual box size=0.5 0.2 0.01
Joints:
- added joint left_arm_pitch: type continuous, parent left_arm_x, child left_arm_y, origin xyz=0 0 0, axis 0 1 0
- added joint left_arm_roll: type continuous, parent base_link, child left_arm_x, origin xyz=-0.2 0 0.2, axis 1 0 0
- added joint left_arm_yaw: type continuous, parent left_arm_y, child left_arm_z, origin xyz=0 0 0, axis 0 0 1
- added joint right_arm_pitch: type continuous, parent right_arm_x, child right_arm_y, origin xyz=0 0 0, axis 0 1 0
- added joint right_arm_roll: type continuous, parent base_link, child right_arm_x, origin xyz=0.2 0 0.2, axis 1 0 0
- added joint right_arm_yaw: type continuous, parent right_arm_y, child right_arm_z, origin xyz=0 0 0, axis 0 0 1
- joint base_to_left_arm: origin xyz=-0.25 0 0 -> xyz=0 0 0; parent base_link -> left_arm_z
- joint base_to_right_arm: origin xyz=0.25 0 0 -> xyz=0 0 0; parent base_link -> right_arm_z
